File: hardware/T12_Control.kicad_sch (KiCad schematic)
At the start: 0 parts

Commit message: Enter schematics for T12 solder iron controller.
Parts:
- added C1, C10, C11, C2, C3, C4, C6, C7, C8, C9: 100nF, Capacitor_SMD:C_0603_1608Metric, symbol Device:C
- added C5: 6.3uF, Capacitor_SMD:C_0603_1608Metric, symbol Device:C
- added D1: RS1M, Diode_SMD:D_SMA, symbol Device:D
- added D2: RED, LED_SMD:LED_0603_1608Metric, symbol Device:LED
- added J1: Screw_Terminal_01x02, PrntrBoardV2:TerminalBlock_Phoenix_PT-1,5-2-3.5-H_1x02_P3.50mm_Horizontal, symbol Connector:Screw_Terminal_01x02
- added J2: GX12-5M, symbol Connector:DIN-5
- added J3: Conn_01x07_Female, Connector_PinSocket_2.54mm:PinSocket_1x07_P2.54mm_Vertical, symbol Connector:Conn_01x07_Female
- added J4: Conn_01x04_Female, Connector_PinSocket_2.54mm:PinSocket_1x04_P2.54mm_Vertical, symbol Connector:Conn_01x04_Female
- added J5: Conn_01x06_Male, Connector_PinHeader_2.54mm:PinHeader_1x06_P2.54mm_Vertical, symbol Connector:Conn_01x06_Male
- added J6: Conn_01x04_Male, Connector_PinHeader_2.54mm:PinHeader_1x04_P2.54mm_Vertical, symbol Connector:Conn_01x04_Male
- added Q1: TPC8107, Package_SO:SO-8_5.3x6.2mm_P1.27mm, symbol TPC8107:TPC8107
- added Q2: SI2308A, Package_TO_SOT_SMD:SOT-23, symbol Device:Q_NMOS_GSD
- added R1: 2k, Resistor_SMD:R_0603_1608Metric, symbol Device:R
- added R2, R7: 10k, Resistor_SMD:R_0603_1608Metric, symbol Device:R
- added R3, R4: 1k, Resistor_SMD:R_0603_1608Metric, symbol Device:R
- added R5: 1k 0.1%, Resistor_SMD:R_0603_1608Metric, symbol Device:R
- added R6: 249k 0.1%, Resistor_SMD:R_0603_1608Metric, symbol Device:R
- added RN1, RN2: 4x4.7k, Resistor_SMD:R_Array_Concave_4x0402, symbol Device:R_Pack04
- added U1: LF15_TO252, Package_TO_SOT_SMD:TO-252-2, symbol Regulator_Linear:LF15_TO252
- added U2: 24LC32, Package_SO:SOIC-8_3.9x4.9mm_P1.27mm, symbol Memory_EEPROM:24LC32
- added U3: SGM8551XN, Package_TO_SOT_SMD:SOT-23-5, symbol Amplifier_Operational:MCP6001-OT
- added U4: STM32F103CBTx, Package_QFP:LQFP-48_7x7mm_P0.5mm, symbol MCU_ST_STM32F1:STM32F103CBTx
Connections:
- new net: Q1.4 (G), R1.2, R3.1
- new net: D1.1 (K), J2.5, Q1.5 (D), Q1.6 (D), Q1.7 (D), Q1.8 (D), RN1.5 (R4.2)
- new net: Q2.2 (S), R3.2
- new net: D2.2 (A), RN1.4 (R4.1), U3.3 (+)
- new net: R5.1, R6.1, U3.4 (-)
- new net: J2.1, RN1.6 (R3.2), RN1.7 (R2.2)
- new net 24V: C1.1, C2.1, J1.2 (Pin_2), Q1.1 (S), Q1.2 (S), Q1.3 (S), R1.1, R2.1, U1.1 (VI)
- new net 3.3V: C10.1, C3.1, C5.1, C6.1, C7.1, C8.1, C9.1, J3.6 (Pin_6), J4.4 (Pin_4), J5.5 (Pin_5), J6.1 (Pin_1), R7.1, RN1.2 (R2.1), RN2.1 (R1.1), RN2.2 (R2.1), RN2.3 (R3.1), RN2.4 (R4.1), U1.3 (VO), U2.8 (VCC), U3.5 (V+), U4.1 (VBAT), U4.24 (VDD), U4.36 (VDD), U4.48 (VDD), U4.9 (VDDA)
- new net ADC2: U4.13 (PA3)
- new net D/~C: J3.2 (Pin_2), U4.26 (PB13)
- new net EE_SCL: RN2.6 (R3.2), U2.6 (SCL), U4.21 (PB10)
- new net EE_SDA: RN2.5 (R4.2), U2.5 (SDA), U4.22 (PB11)
- new net GND: C1.2, C10.2, C11.1, C2.2, C3.2, C4.2, C5.2, C6.2, C7.2, C8.2, C9.2, D1.2 (A), D2.1 (K), J1.1 (Pin_1), J2.3, J2.4, J3.7 (Pin_7), J4.3 (Pin_3), J5.6 (Pin_6), J6.2 (Pin_2), Q2.3 (D), R4.2, R5.2, U1.2 (GND), U2.1 (A0), U2.2 (A1), U2.3 (A2), U2.4 (GND), U2.7 (WP), U3.2 (V-), U4.23 (VSS), U4.35 (VSS), U4.44 (BOOT0), U4.47 (VSS), U4.8 (VSSA)
- new net HEARER_ON: Q2.1 (G)
- new net HEATER_ON: U4.29 (PA8)
- new net IO_1: U4.2 (PC13)
- new net IO_2: U4.3 (PC14)
- new net IO_3: U4.4 (PC15)
- new net MISO: U4.16 (PA6)
- new net MOSI: J3.4 (Pin_4), U4.17 (PA7)
- new net NTC: RN1.3 (R3.1), U4.12 (PA2)
- new net OLED_SCL: J4.2 (Pin_2), RN2.8 (R1.2), U4.45 (PB8)
- new net OLED_SDA: J4.1 (Pin_1), RN2.7 (R2.2), U4.46 (PB9)
- new net PWM1: U4.38 (PA15)
- new net PWM2: U4.18 (PB0)
- new net PWM3: U4.19 (PB1)
- new net RX: J6.3 (Pin_3), U4.31 (PA10)
- new net SCK: J3.5 (Pin_5), U4.15 (PA5)
- new net SHAKE: J2.2
- new net SWDCLK: J5.2 (Pin_2), U4.37 (PA14)
- new net SWDIO: J5.3 (Pin_3), U4.34 (PA13)
- new net SWDSWO: J5.1 (Pin_1), U4.39 (PB3)
- new net TIP_TEMP: R6.2, U3.1, U4.10 (PA0)
- new net TX: J6.4 (Pin_4), U4.30 (PA9)
- new net V_MON: C4.1, R2.2, R4.1, U4.11 (PA1)
- new net ~CS: J3.1 (Pin_1), U4.20 (PB2)
- new net ~NRST: C11.2, J5.4 (Pin_4), R7.2, U4.7 (NRST)
- new net ~RST: J3.3 (Pin_3), U4.25 (PB12)
Other:
- note added: "2.25V=450C"
- note added: "D/C"
- note added: "GND"
- note added: "SCL"
- note added: "SDA"
- note added: "VCC"
- note added: "~CS"
- note added: "~RST"
