File: hardware/ToolBoard.kicad_sch (KiCad schematic)
At the start: 0 parts

Commit message: Added endstops, adc, pwm, dirver and power.
Parts:
- added C? (x2): 10uF, PrntrBoardV2:C_0603_1608Metric, symbol Device:C
- added C? (x7): 1000pF, PrntrBoardV2:C_0603_1608Metric, symbol Device:C
- added C? (x5): 0.1uF, PrntrBoardV2:C_0603_1608Metric, symbol Device:C
- added C? (x2): 0.1uF 50V, PrntrBoardV2:C_0402_1005Metric, symbol Device:C
- added C? (x3): 10uF 50V, PrntrBoardV2:C_1206_3216Metric, symbol Device:C
- added C?: 0.022uF 50V, PrntrBoardV2:C_0603_1608Metric, symbol Device:C
- added C?: 2.2uF, PrntrBoardV2:C_0603_1608Metric, symbol Device:C
- added C?: 100uV 35V, Capacitor_SMD:CP_Elec_6.3x7.7, symbol Device:CP
- added D? (x7): LED, PrntrBoardV2:LED_0603_1608Metric, symbol Device:LED
- added D? (x3): B5819W, Diode_SMD:D_SOD-123, symbol Device:D_Schottky
- added D? (x2): 1N4148, Diode_SMD:D_SOD-323_HandSoldering, symbol Device:D
- added D?: BAT54S, Package_TO_SOT_SMD:SOT-23, symbol Device:D_Schottky_x2_Serial_AKC
- added F?: Fuse, PrntrBoardV2:2410_FuseFolder, symbol Device:Fuse
- added F?: 500mA, PrntrBoardV2:R_0603_1608Metric, symbol Device:Polyfuse
- added H? (x4): MountingHole, MountingHole:MountingHole_3.2mm_M3, symbol Mechanical:MountingHole
- added H? (x2): JLC Tooling Hole, PrntrBoardV2:JLC_Tool_hole, symbol Mechanical:MountingHole
- added J? (x2): JST XH, Connector_JST:JST_XH_B2B-XH-A_1x02_P2.50mm_Vertical, symbol Connector:Screw_Terminal_01x02
- added J?: USB_B_Micro, PrntrBoardV2:MC-101C, symbol Connector:USB_B_Micro
- added J? (x2): KF350, PrntrBoardV2:TerminalBlock_Phoenix_PT-1,5-2-3.5-H_1x02_P3.50mm_Horizontal, symbol Connector:Screw_Terminal_01x02
- added J?: Conn_01x04_Male, PrntrBoardV2:Molex-SL-4POS, symbol Connector:Conn_01x04_Male
- added J? (x2), J_TH?: JST XH, Connector_JST:JST_XH_B2B-XH-A_1x02_P2.50mm_Vertical, symbol Connector_Generic:Conn_02x01
- added JP?: Jumper_3_Open, Connector_PinHeader_2.54mm:PinHeader_1x03_P2.54mm_Vertical, symbol Jumper:Jumper_3_Open
- added J_SER?: Serial 0, Connector_PinHeader_2.54mm:PinHeader_1x04_P2.54mm_Vertical, symbol Connector:Conn_01x04_Male
- added J_SWD?: SWD, Connector_PinHeader_2.54mm:PinHeader_1x05_P2.54mm_Vertical, symbol Connector:Conn_01x05_Male
- added J_X-? (x2): JST XH 3p, Connector_JST:JST_XH_B3B-XH-A_1x03_P2.50mm_Vertical, symbol Connector:Conn_01x03_Male
- added LOGO?: Logo_Open_Hardware_Small, Symbol:OSHW-Logo2_9.8x8mm_SilkScreen, symbol Graphic:Logo_Open_Hardware_Small
- added R? (x9): 10k, PrntrBoardV2:R_0603_1608Metric, symbol Device:R
- added R? (x4): 470, PrntrBoardV2:R_0603_1608Metric, symbol Device:R
- added R? (x3): 1k, PrntrBoardV2:R_0603_1608Metric, symbol Device:R
- added R?: 100k, PrntrBoardV2:R_0603_1608Metric, symbol Device:R
- added R?: 180, PrntrBoardV2:R_0603_1608Metric, symbol Device:R
- added R? (x2): 22, PrntrBoardV2:R_0603_1608Metric, symbol Device:R
- added R? (x2): 0R091, Resistor_SMD:R_1210_3225Metric, symbol Device:R
- added R?: 1.5k, PrntrBoardV2:R_0603_1608Metric, symbol Device:R
- added R?: 4k7, PrntrBoardV2:R_0603_1608Metric, symbol Device:R
- added TC?: TC, kicad-molex-sl-footprints:Molex-SL-6POS, symbol Connector_Generic:Conn_01x06
- added TR? (x2): SI2318CDS, PrntrBoardV2:SOT-23, symbol bsh105:BSH105
- added TR?: PSMN7R0-30YL, Package_SON:VSON-8_3.3x3.3mm_P0.65mm_NexFET, symbol ipd036n04l:IPD036N04L
- added U?: 74AHCT1G14, Package_TO_SOT_SMD:SOT-23-5, symbol Logic_74xgxx:74AHCT1G14
- added U?: AMS1117-3.3, Package_TO_SOT_SMD:SOT-223-3_TabPin2, symbol Regulator_Linear:AMS1117-3.3
- added U?: TMC2209-LA, PrntrBoardV2:TMC22xx_QFN, symbol tmc2209:TMC2209-LA
Connections:
- new net: D?.2 (A), R?.2 (x7)
- new net: D?.1 (K), D?.2 (A), J?.2 (Pin_2), TR?.D
- new net: D?.2 (A), J?.2 (Pin_2), TR?.D (x2)
- new net: R?.1, TR?.G (x3)
- new net: D?.1 (K), D?.2 (A), R?.2 (x2)
- new net: C?.1, D?.1 (K), J_X-?.1 (Pin_1) (x2)
- new net: F?.1, J?.1 (VBUS)
- new net: C?.2, J?.6 (Shield), R?.2
- new net: F?.1, J?.2 (Pin_2)
- new net: R?.2, U?.4
- new net: C?.2, U?.6 (VCP)
- new net: R?.1, U?.14 (PDN_UART)
- new net: J_TH?.1 (Pin_1), R?.2, R?.2
- new net: R?.2, U?.27 (BRB)
- new net: C?.1, C?.1, U?.28 (VS(B))
- new net: R?.2, U?.23 (BRA)
- new net: C?.2, U?.4 (CPO)
- new net: C?.1, U?.5 (CPI)
- new net: C?.2, U?.8 (5Vout)
- new net 3.3V: C?.1, C?.1, C?.1, J_SWD?.2 (Pin_2), R?.1, R?.1, R?.1, R?.1, R?.2, U?.15 (VCC_IO), U?.2 (VO)
- new net ADC1: C?.1, D?.3 (common), R?.1, TC?.6 (Pin_6)
- new net AVREF: D?.2 (K), R?.1
- new net D+: J?.3 (D+), R?.1, R?.1
- new net D-: J?.2 (D-), R?.1
- new net DIAG: U?.11 (DIAG)
- new net DIR: U?.19 (DIR)
- new net FAN1: R?.1, R?.2
- new net FAN2: R?.1, R?.2
- new net GND: C?.1, C?.1, C?.1, C?.1, C?.1, C?.1, C?.2, C?.2, C?.2, C?.2, C?.2, C?.2, C?.2, C?.2, C?.2, C?.2, C?.2, C?.2, C?.2, C?.2, D?.1 (A), D?.1 (K), D?.1 (K), D?.1 (K), D?.1 (K), J?.1 (Pin_1), J?.2 (Pin_2), J?.2 (Pin_2), J?.5 (GND), J_SER?.2 (Pin_2), J_SWD?.1 (Pin_1), J_TH?.2 (Pin_2), J_X-?.2 (Pin_2), J_X-?.2 (Pin_2), R?.1, R?.1, R?.1, R?.2, R?.2, TC?.1 (Pin_1), TR?.S, TR?.S, TR?.S, U?.1 (GND), U?.10 (MS2), U?.13 (CLK_IN), U?.18 (GND), U?.20 (~STDBY), U?.25 (NC), U?.29 (PAD), U?.3 (GND), U?.3 (GND), U?.9 (MS1)
- new net HEATER: R?.2, U?.2
- new net MOTA1: C?.2, J?.3 (Pin_3), U?.24 (OA1)
- new net MOTA2: C?.2, J?.4 (Pin_4), U?.21 (OA2)
- new net MOTB1: C?.2, J?.2 (Pin_2), U?.26 (OB1)
- new net MOTB2: C?.2, J?.1 (Pin_1), U?.1 (OB2)
- new net SPI1_MISO: TC?.5 (Pin_5)
- new net SPI1_MOSI: TC?.4 (Pin_4)
- new net SPI1_SCK: TC?.3 (Pin_3)
- new net STEP: U?.16 (STEP)
- new net ST_UART: R?.2
- new net SWDCLK: J_SWD?.5 (Pin_5)
- new net SWDIO: J_SWD?.4 (Pin_4)
- new net UART_RX: J_SER?.3 (Pin_3)
- new net UART_TX: J_SER?.4 (Pin_4)
- new net USB_D+: R?.2
- new net USB_D-: R?.2
- new net VCC: C?.1, C?.1, F?.2, J?.1 (Pin_1), JP?.1 (A), J_SER?.1 (Pin_1), J_X-?.3 (Pin_3), J_X-?.3 (Pin_3), R?.1, TC?.2 (Pin_2), U?.3 (VI), U?.5 (VCC)
- new net V_fan: D?.1 (K), D?.1 (K), J?.1 (Pin_1), J?.1 (Pin_1), JP?.2 (C), R?.1
- new net V_motors: C?.1, C?.1, C?.1, C?.1, C?.1, D?.1 (K), F?.2, J?.1 (Pin_1), J?.1 (Pin_1), JP?.3 (B), R?.1, R?.1, U?.22 (VS(A))
- new net ~ENABLE: U?.2 (~ENN)
- new net ~E_STOP1: R?.1
- new net ~E_STOP2: R?.1
- new net ~RESET: J_SWD?.3 (Pin_3)
- no-connect marks 0 -> 4
Other:
- note added: "1%"
- note added: "5A"
