File: hardware/ToolBoard.kicad_sch (KiCad schematic)
At the start: 89 parts

Commit message: Update toolboard.
Parts:
- removed D? (x2): B5819W, Diode_SMD:D_SOD-123, symbol Device:D_Schottky
- removed J? (x2): JST XH, Connector_JST:JST_XH_B2B-XH-A_1x02_P2.50mm_Vertical, symbol Connector_Generic:Conn_02x01
- removed JP?: Jumper_3_Open, Connector_PinHeader_2.54mm:PinHeader_1x03_P2.54mm_Vertical, symbol Jumper:Jumper_3_Open
- removed J_SER?: Serial 0, Connector_PinHeader_2.54mm:PinHeader_1x04_P2.54mm_Vertical, symbol Connector:Conn_01x04_Male
- removed J_SWD?: SWD, Connector_PinHeader_2.54mm:PinHeader_1x05_P2.54mm_Vertical, symbol Connector:Conn_01x05_Male
- added C1, C2: 22pF, Capacitor_SMD:C_0402_1005Metric, symbol Device:C
- added C3: 0.1uF, PrntrBoardV2:C_0603_1608Metric, symbol Device:C
- added D11, D6: 1N4148, Diode_SMD:D_SOD-323_HandSoldering, symbol Device:D
- added J1: DBG, Connector_PinHeader_1.27mm:PinHeader_2x04_P1.27mm_Vertical, symbol Connector_Generic:Conn_02x04_Odd_Even
- added R1, R2: 10k, PrntrBoardV2:R_0603_1608Metric, symbol Device:R
- added R8: 1k, PrntrBoardV2:R_0603_1608Metric, symbol Device:R
- added SW_BOOT1: SW_Push, PrntrBoardV2:Button_4x4, symbol Switch:SW_Push
- added U2: STM32F103C8Tx, Package_QFP:LQFP-48_7x7mm_P0.5mm, symbol MCU_ST_STM32F1:STM32F103C8Tx
- added Y1: 8MHz, Crystal:Crystal_SMD_5032-2Pin_5.0x3.2mm, symbol Device:Crystal
- F1: renamed from F?; footprint PrntrBoardV2:2410_FuseFolder -> Fuse:Fuse_1206_3216Metric; LCSC Part # (none) -> C163128; Part # (none) -> CFS12V3T5R0
- H1, H2, H3, H4: renamed from H?; footprint MountingHole:MountingHole_3.2mm_M3 -> MountingHole:MountingHole_3.2mm_M3_Pad_Via
- J2: renamed from J?; footprint PrntrBoardV2:Molex-SL-4POS -> Connector_JST:JST_PH_B4B-PH-K_1x04_P2.00mm_Vertical
- J4, J8: renamed from J?; footprint PrntrBoardV2:TerminalBlock_Phoenix_PT-1,5-2-3.5-H_1x02_P3.50mm_Horizontal -> TerminalBlock_Phoenix:TerminalBlock_Phoenix_MPT-0,5-2-2.54_1x02_P2.54mm_Horizontal
- J5, J6: renamed from J?; footprint Connector_JST:JST_XH_B2B-XH-A_1x02_P2.50mm_Vertical -> Connector_JST:JST_PH_B2B-PH-K_1x02_P2.00mm_Vertical
- J_TH1: renamed from J_TH?; footprint Connector_JST:JST_XH_B2B-XH-A_1x02_P2.50mm_Vertical -> Connector_JST:JST_PH_B2B-PH-K_1x02_P2.00mm_Vertical
- J_X-1, J_X-2: renamed from J_X-?; footprint Connector_JST:JST_XH_B3B-XH-A_1x03_P2.50mm_Vertical -> Connector_JST:JST_PH_B3B-PH-K_1x03_P2.00mm_Vertical
- TR3: renamed from TR?; footprint Package_SON:VSON-8_3.3x3.3mm_P0.65mm_NexFET -> PrntrBoardV2:VSON-8_3.3x3.3mm_P0.65mm_NexFET
- gave numbers to parts that had none: 68
Connections:
- net 3.3V: now also J1.8 (Pin_8), R8.1
- net ADC1: now also U2.10 (PA0)
- net D+: now also U2.33 (PA12)
- net D-: now also U2.32 (PA11)
- net FAN1: now also U2.21 (PB10)
- net FAN2: now also U2.22 (PB11)
- net GND: now also C1.1, C2.1, C3.2, J1.7 (Pin_7), R1.2; no longer C5.2
- net HEATER: now also U2.46 (PB9)
- net ST_UART: now also U2.12 (PA2)
- net SWDCLK: now also J1.2 (Pin_2), U2.37 (PA14)
- net SWDIO: now also J1.4 (Pin_4), U2.34 (PA13)
- net UART_RX: now also J1.1 (Pin_1), U2.31 (PA10)
- net UART_TX: now also J1.3 (Pin_3), U2.30 (PA9)
- net V_fan: no longer J5.1 (Pin_1), J6.1 (Pin_1)
- net V_motors: now also J5.1 (Pin_1), J6.1 (Pin_1), D11.1 (K), D6.1 (K)
- net at J6.2 (Pin_2), TR2.D: now also D11.2 (A)
- net at J5.2 (Pin_2), TR1.D: now also D6.2 (A)
- new net: C1.2, U2.5 (PD0), Y1.2
- new net: R1.1, U2.44 (BOOT0)
- new net: C2.2, U2.6 (PD1), Y1.1
- new net: R8.2, SW_BOOT1.1
- new net BOOT: J1.5 (Pin_5), SW_BOOT1.2
- new net MISO: U2.16 (PA6)
- new net MOSI: U2.17 (PA7)
- new net SCK: U2.15 (PA5)
- new net SCL: U2.42 (PB6)
- new net SDA: U2.43 (PB7)
- new net ~RST: C3.1, J1.6 (Pin_6), R2.2, U2.7 (NRST)
Other:
- note added: "BOOT"
- moved on the sheet: J5, J6, R17, R18, TR2
