File: hardware/ToolBoard.kicad_pcb (KiCad board)
At the start: 0 parts

Commit message: Update toolboard.
Parts:
- added C1: 22pF, Capacitor_SMD:C_0402_1005Metric, F.Cu at (105.5, 138.6)
- added C10: 0.022uF 50V, PrntrBoardV2:C_0603_1608Metric, F.Cu at (89.6, 103.7)
- added C11: 0.1uF, PrntrBoardV2:C_0603_1608Metric, F.Cu at (142.7, 76.8)
- added C12: 0.1uF 50V, PrntrBoardV2:C_0402_1005Metric, F.Cu at (109.0, 122.0)
- added C13: 0.1uF 50V, PrntrBoardV2:C_0402_1005Metric, F.Cu at (112.8, 104.5)
- added C14: 10uF 50V, PrntrBoardV2:C_1206_3216Metric, F.Cu at (148.0, 60.9)
- added C15: 10uF 50V, PrntrBoardV2:C_1206_3216Metric, F.Cu at (127.5, 82.6)
- added C16: 1000pF, PrntrBoardV2:C_0603_1608Metric, F.Cu at (138.7, 77.9)
- added C17: 1000pF, PrntrBoardV2:C_0603_1608Metric, F.Cu at (161.7, 62.2)
- added C18: 1000pF, PrntrBoardV2:C_0603_1608Metric, F.Cu at (145.3, 72.5)
- added C19: 1000pF, PrntrBoardV2:C_0603_1608Metric, F.Cu at (149.4, 70.0)
- added C2: 22pF, Capacitor_SMD:C_0402_1005Metric, F.Cu at (105.5, 141.4)
- added C20: 100uV 35V, Capacitor_SMD:CP_Elec_6.3x7.7, F.Cu at (126.1, 130.8)
- added C21: 1000pF, PrntrBoardV2:C_0603_1608Metric, F.Cu at (113.3, 102.3)
- added C22: 1000pF, PrntrBoardV2:C_0603_1608Metric, F.Cu at (132.3, 82.2)
- added C23: 1000pF, PrntrBoardV2:C_0603_1608Metric, F.Cu at (136.3, 83.0)
- added C24: 10uF 50V, PrntrBoardV2:C_1206_3216Metric, F.Cu at (135.6, 75.0)
- added C25: 0.1uF, PrntrBoardV2:C_0603_1608Metric, F.Cu at (145.3, 70.0)
- added C3: 0.1uF, PrntrBoardV2:C_0603_1608Metric, F.Cu at (134.7, 78.0)
- added C4: 10uF, PrntrBoardV2:C_0603_1608Metric, F.Cu at (161.8, 59.7)
- added C5: 0.1uF, PrntrBoardV2:C_0603_1608Metric, F.Cu at (146.7, 77.5)
- added C6: 0.1uF, PrntrBoardV2:C_0603_1608Metric, F.Cu at (153.6, 67.0)
- added C7: 10uF, PrntrBoardV2:C_0603_1608Metric, F.Cu at (126.5, 95.3)
- added C8: 0.1uF, PrntrBoardV2:C_0603_1608Metric, F.Cu at (103.7, 69.4)
- added C9: 2.2uF, PrntrBoardV2:C_0603_1608Metric, F.Cu at (157.8, 59.7)
- added D1: LED, PrntrBoardV2:LED_0603_1608Metric, F.Cu at (149.7, 67.2)
- added D10: LED, PrntrBoardV2:LED_0603_1608Metric, F.Cu at (127.8, 92.7)
- added D11: 1N4148, Diode_SMD:D_SOD-323_HandSoldering, F.Cu at (138.3, 103.6)
- added D12: LED, PrntrBoardV2:LED_0603_1608Metric, F.Cu at (152.8, 61.9)
- added D13: B5819W, Diode_SMD:D_SOD-123, F.Cu at (148.1, 57.6)
- added D2: LED, PrntrBoardV2:LED_0603_1608Metric, F.Cu at (149.7, 64.5)
- added D3: LED, PrntrBoardV2:LED_0603_1608Metric, F.Cu at (141.4, 71.7)
- added D4: LED, PrntrBoardV2:LED_0603_1608Metric, F.Cu at (127.8, 90.1)
- added D5: 1N4148, Diode_SMD:D_SOD-323_HandSoldering, F.Cu at (94.5, 65.1)
- added D6: 1N4148, Diode_SMD:D_SOD-323_HandSoldering, F.Cu at (143.3, 103.6)
- added D7: BAT54S, Package_TO_SOT_SMD:SOT-23, F.Cu at (97.4, 130.7)
- added D8: LED, PrntrBoardV2:LED_0603_1608Metric, F.Cu at (123.8, 90.9)
- added D9: 1N4148, Diode_SMD:D_SOD-323_HandSoldering, F.Cu at (94.5, 68.1)
- added F1: Fuse, Fuse:Fuse_1206_3216Metric, F.Cu at (128.3, 126.0)
- added F2: 500mA, PrntrBoardV2:R_0603_1608Metric, F.Cu at (131.8, 90.5)
- added H1: MountingHole, MountingHole:MountingHole_3.2mm_M3_Pad_Via, F.Cu at (93.0, 149.0)
- added H2: MountingHole, MountingHole:MountingHole_3.2mm_M3_Pad_Via, F.Cu at (127.0, 149.0)
- added H3: MountingHole, MountingHole:MountingHole_3.2mm_M3_Pad_Via, F.Cu at (127.0, 115.0)
- added H4: MountingHole, MountingHole:MountingHole_3.2mm_M3_Pad_Via, F.Cu at (93.0, 115.0)
- added J1: DBG, Connector_PinHeader_1.27mm:PinHeader_2x04_P1.27mm_Vertical, F.Cu at (116.0, 151.3)
- added J2: Conn_01x04_Male, Connector_JST:JST_PH_B4B-PH-K_1x04_P2.00mm_Vertical, F.Cu at (118.4, 114.0)
- added J4: KF350, TerminalBlock_Phoenix:TerminalBlock_Phoenix_MPT-0,5-2-2.54_1x02_P2.54mm_Horizontal, F.Cu at (127.7, 122.8)
- added J5: JST XH, Connector_JST:JST_PH_B2B-PH-K_1x02_P2.00mm_Vertical, F.Cu at (93.1, 126.7)
- added J6: JST XH, Connector_JST:JST_PH_B2B-PH-K_1x02_P2.00mm_Vertical, F.Cu at (93.1, 121.4)
- added J7: USB_B_Micro, PrntrBoardV2:MC-101C, F.Cu at (128.7, 140.4)
- added J8: KF350, TerminalBlock_Phoenix:TerminalBlock_Phoenix_MPT-0,5-2-2.54_1x02_P2.54mm_Horizontal, F.Cu at (92.5, 136.0)
- added J_TH1: JST XH, Connector_JST:JST_PH_B2B-PH-K_1x02_P2.00mm_Vertical, F.Cu at (93.1, 131.9)
- added J_X-1: JST XH 3p, Connector_JST:JST_PH_B3B-PH-K_1x03_P2.00mm_Vertical, F.Cu at (102.6, 151.2)
- added J_X-2: JST XH 3p, Connector_JST:JST_PH_B3B-PH-K_1x03_P2.00mm_Vertical, F.Cu at (111.2, 151.2)
- added LOGO1: Logo_Open_Hardware_Small, Symbol:OSHW-Logo2_9.8x8mm_SilkScreen, F.Cu at (94.4, 90.4)
- added R1: 10k, PrntrBoardV2:R_0603_1608Metric, F.Cu at (140.3, 82.9)
- added R10: 1k, PrntrBoardV2:R_0603_1608Metric, F.Cu at (153.6, 69.5)
- added R11: 10k, PrntrBoardV2:R_0603_1608Metric, F.Cu at (157.8, 57.2)
- added R12: 1k, PrntrBoardV2:R_0603_1608Metric, F.Cu at (161.8, 57.2)
- added R13: 4k7, PrntrBoardV2:R_0603_1608Metric, F.Cu at (131.1, 85.5)
- added R14: 10k, PrntrBoardV2:R_0603_1608Metric, F.Cu at (117.4, 103.7)
- added R15: 470, PrntrBoardV2:R_0603_1608Metric, F.Cu at (135.8, 88.0)
- added R16: 10k, PrntrBoardV2:R_0603_1608Metric, F.Cu at (131.8, 88.0)
- added R17: 10k, PrntrBoardV2:R_0603_1608Metric, F.Cu at (118.5, 98.7)
- added R18: 1k, PrntrBoardV2:R_0603_1608Metric, F.Cu at (140.3, 80.4)
- added R19: 10k, PrntrBoardV2:R_0603_1608Metric, F.Cu at (146.7, 75.0)
- added R2: 10k, PrntrBoardV2:R_0603_1608Metric, F.Cu at (136.3, 80.5)
- added R20: 470, PrntrBoardV2:R_0603_1608Metric, F.Cu at (137.3, 71.7)
- added R21: 10k, PrntrBoardV2:R_0603_1608Metric, F.Cu at (157.7, 64.7)
- added R22: 180, PrntrBoardV2:R_0603_1608Metric, F.Cu at (122.5, 96.7)
- added R23: 10k, PrntrBoardV2:R_0603_1608Metric, F.Cu at (140.4, 74.3)
- added R24: 1.5k, PrntrBoardV2:R_0603_1608Metric, F.Cu at (149.4, 72.5)
- added R25: 22, PrntrBoardV2:R_0603_1608Metric, F.Cu at (122.5, 99.2)
- added R26: 22, PrntrBoardV2:R_0603_1608Metric, F.Cu at (114.5, 98.7)
- added R27: 100k, PrntrBoardV2:R_0603_1608Metric, F.Cu at (135.8, 85.5)
- added R3: 470, PrntrBoardV2:R_0603_1608Metric, F.Cu at (157.7, 62.2)
- added R4: 0R091, Resistor_SMD:R_1210_3225Metric, F.Cu at (119.0, 118.0)
- added R5: 0R091, Resistor_SMD:R_1210_3225Metric, F.Cu at (111.0, 118.0)
- added R6: 10k, PrntrBoardV2:R_0603_1608Metric, F.Cu at (117.4, 101.2)
- added R7: 10k, PrntrBoardV2:R_0603_1608Metric, F.Cu at (93.6, 103.7)
- added R8: 1k, PrntrBoardV2:R_0603_1608Metric, F.Cu at (122.5, 94.2)
- added R9: 470, PrntrBoardV2:R_0603_1608Metric, F.Cu at (153.6, 64.5)
- added SW_BOOT1: SW_Push, PrntrBoardV2:Button_4x4, F.Cu at (122.4, 77.1)
- added TC1: TC, kicad-molex-sl-footprints:Molex-SL-6POS, F.Cu at (87.1, 60.3)
- added TH1: JLC Tooling Hole, PrntrBoardV2:JLC_Tool_hole, F.Cu at (105.0, 71.7)
- added TH2: JLC Tooling Hole, PrntrBoardV2:JLC_Tool_hole, F.Cu at (105.0, 73.9)
- added TR1: SI2318CDS, PrntrBoardV2:SOT-23, F.Cu at (126.9, 86.5)
- added TR2: SI2318CDS, PrntrBoardV2:SOT-23, F.Cu at (109.1, 103.3)
- added TR3: PSMN7R0-30YL, PrntrBoardV2:VSON-8_3.3x3.3mm_P0.65mm_NexFET, F.Cu at (98.4, 138.6)
- added U1: AMS1117-3.3, Package_TO_SOT_SMD:SOT-223-3_TabPin2, F.Cu at (123.2, 60.0)
- added U2: STM32F103C8Tx, Package_QFP:LQFP-48_7x7mm_P0.5mm, F.Cu at (117.0, 141.0)
- added U3: TMC2209-LA, PrntrBoardV2:TMC22xx_QFN, F.Cu at (115.0, 123.0)
- added U4: 74AHCT1G14, Package_TO_SOT_SMD:SOT-23-5, F.Cu at (153.3, 58.2)
- added Y1: 8MHz, Crystal:Crystal_SMD_5032-2Pin_5.0x3.2mm, F.Cu at (108.0, 140.0)
Other:
- board outline added: 42 x 42 mm
- copper layers 0 -> 2
